Commit message: Add some dependent packages

File: models/Inverted_pendulum/Inverted_pendulum.xacro (robot description, xacro)
@@ -17,5 +17,5 @@
     <!-- links and joints -->
     <link name="base_link"/>
-    <joint name="base_joint" type="fixed">
+    <joint name="cart_joint" type="fixed">
         <origin xyz="0.0 0.0 ${cart_height/2}" rpy="0.0 0.0 0.0"/>
         <parent link="base_link"/>

Commit message: Add link effort plugin for inverted pendulum sim

File: models/Inverted_pendulum/Inverted_pendulum.xacro (robot description, xacro)
@@ -16,11 +16,6 @@
     <xacro:include filename="$(find robot_sim_cpp)/models/Inverted_pendulum/Inverted_pendulum.gazebo"/>
     <!-- links and joints -->
-    <link name="base_link"/>
-    <joint name="cart_joint" type="fixed">
-        <origin xyz="0.0 0.0 ${cart_height/2}" rpy="0.0 0.0 0.0"/>
-        <parent link="base_link"/>
-        <child link="cart_link"/>
-    </joint>
     <link name="cart_link">
+        <pose>0 0 ${cart_height/2} 0 0 0</pose>
         <inertial>
             <mass value="${cart_mass}"/>
@@ -36,12 +31,20 @@
                 <box size="${cart_depth} ${cart_width} ${cart_height}"/>
             </geometry>
+            <surface>
+                <friction>
+                    <ode>
+                        <mu>${friction_coefficient}</mu>
+                        <mu2>${friction_coefficient}</mu2>
+                    </ode>
+                </friction>
+            </surface>
         </collision>
     </link>
     <joint name="pendulum_joint" type="revolute">
-        <origin xyz="0.0 0.0 ${cart_height + pendulum_radius}" rpy="0.0 0.0 0.0"/>
-        <parent link="base_link"/>
+        <origin xyz="0.0 0.0 ${cart_height/2 + pendulum_radius}" rpy="0.0 0.0 0.0"/>
+        <parent link="cart_link"/>
         <child link="pendulum_link"/>
         <axis xyz="0.0 -1.0 0.0"/>
-        <limit lower="${-PI}" upper="${PI}" effort="0.0" velocity="0.0"/>
+        <limit lower="${-PI/2}" upper="${PI/2}" effort="0.0" velocity="0.0"/>
     </joint>
     <link name="pendulum_link">

Commit message: Get pendulum parameters from user

File: models/Inverted_pendulum/Inverted_pendulum.xacro (robot description, xacro)
@@ -1,15 +1,21 @@
 <?xml version="1.0"?>
 <robot name="Inverted_pendulum" xmlns:xacro="http://www.ros.org/wiki/xacro">
+    <!-- arguments -->
+    <xacro:arg name="cart_mass" default="0.5"/>
+    <xacro:arg name="pendulum_mass" default="0.2"/>
+    <xacro:arg name="friction_coefficient" default="0.1"/>
+    <xacro:arg name="length_to_COM" default="0.3"/>
+    <xacro:arg name="pendulum_mass_moment" default="0.006"/>
     <!-- properties -->
     <xacro:property name="PI" value="3.141593"/>
-    <xacro:property name="cart_mass" value="0.5"/>
-    <xacro:property name="pendulum_mass" value="0.2"/>
-    <xacro:property name="friction_coefficient" value="0.1"/>
-    <xacro:property name="length_to_COM" value="0.3"/>
-    <xacro:property name="pendulum_mass_moment" value="0.006"/>
+    <xacro:property name="cart_mass" value="$(arg cart_mass)"/>
+    <xacro:property name="pendulum_mass" value="$(arg pendulum_mass)"/>
+    <xacro:property name="friction_coefficient" value="$(arg friction_coefficient)"/>
+    <xacro:property name="length_to_COM" value="$(arg length_to_COM)"/>
+    <xacro:property name="pendulum_mass_moment" value="$(arg pendulum_mass_moment)"/>
     <xacro:property name="cart_width" value="0.5"/>
     <xacro:property name="cart_depth" value="1.0"/>
     <xacro:property name="cart_height" value="0.5"/>
-    <xacro:property name="pendulum_length" value="0.6"/>
+    <xacro:property name="pendulum_length" value="$(eval length_to_COM * 2)"/>
     <xacro:property name="pendulum_radius" value="0.03"/>
     <!-- include -->
